Commit message: added casadi wrapper for gpu IK

File: Go2_pinocchio/go2.urdf (robot description, URDF)
Before this commit: robot go2_description, 42 links, 41 joints
Joints:
- joint FL_thigh_joint: limit lower=-1.5708 upper=3.4907 effort=23.7 velocity=30.1 -> lower=-3.4907 upper=3.4907 effort=23.7 velocity=30.1
- joint FR_thigh_joint: limit lower=-1.5708 upper=3.4907 effort=23.7 velocity=30.1 -> lower=-3.4907 upper=3.4907 effort=23.7 velocity=30.1

File: Go2_pinocchio/go2_original.urdf (robot description, URDF)
Before this commit: robot go2_corrected_fixed3, 44 links, 43 joints
Links:
- removed link floor
- link FL_calf: geometry collision cylinder length=0.12 radius=0.012; visual mesh filename=package://go2_description/dae/calf.dae
- link FL_foot: geometry collision sphere radius=0.022; visual mesh filename=package://go2_description/dae/foot.dae
- link FL_hip: geometry collision cylinder length=0.04 radius=0.046; visual mesh filename=package://go2_description/dae/hip.dae
- link FL_thigh: geometry collision box size=0.213 0.0245 0.034; visual mesh filename=package://go2_description/dae/thigh.dae
- link FR_calf: geometry collision cylinder length=0.12 radius=0.013; visual mesh filename=package://go2_description/dae/calf_mirror.dae
- link FR_foot: geometry collision sphere radius=0.022; visual mesh filename=package://go2_description/dae/foot.dae
- link FR_hip: geometry collision cylinder length=0.04 radius=0.046; visual mesh filename=package://go2_description/dae/hip.dae
- link FR_thigh: geometry collision box size=0.213 0.0245 0.034; visual mesh filename=package://go2_description/dae/thigh_mirror.dae
- link RL_calf: geometry collision cylinder length=0.12 radius=0.013; visual mesh filename=package://go2_description/dae/calf.dae
- link RL_foot: geometry collision sphere radius=0.022; visual mesh filename=package://go2_description/dae/foot.dae
- link RL_hip: geometry collision cylinder length=0.04 radius=0.046; visual mesh filename=package://go2_description/dae/hip.dae
- link RL_thigh: geometry collision box size=0.213 0.0245 0.034; visual mesh filename=package://go2_description/dae/thigh.dae
- link RR_calf: geometry collision cylinder length=0.12 radius=0.013; visual mesh filename=package://go2_description/dae/calf_mirror.dae
- link RR_foot: geometry collision sphere radius=0.022; visual mesh filename=package://go2_description/dae/foot.dae
- link RR_hip: geometry collision cylinder length=0.04 radius=0.046; visual mesh filename=package://go2_description/dae/hip.dae
- link RR_thigh: geometry collision box size=0.213 0.0245 0.034; visual mesh filename=package://go2_description/dae/thigh_mirror.dae
- link base: geometry collision box size=0.3762 0.0935 0.114; visual mesh filename=package://go2_description/dae/base.dae
Joints:
- removed joint floor_to_world
- removed joint world_to_base
- added joint world_to_base_fixed: type fixed, parent world, child base, origin xyz=0 0 0.445 rpy=0 0 0
- joint FL_calf_joint: axis 0 -1 0 -> 0 1 0
- joint FL_thigh_joint: axis 0 -1 0 -> 0 1 0; limit lower=-3.4907 upper=1.5708 effort=23.7 velocity=30.1 -> lower=-1.5708 upper=3.4907 effort=23.7 velocity=30.1
- joint FR_calf_joint: axis 0 -1 0 -> 0 1 0
- joint FR_thigh_joint: axis 0 -1 0 -> 0 1 0; limit lower=-3.4907 upper=1.5708 effort=23.7 velocity=30.1 -> lower=-1.5708 upper=3.4907 effort=23.7 velocity=30.1
- joint RL_calf_joint: axis 0 -1 0 -> 0 1 0
- joint RL_thigh_joint: axis 0 -1 0 -> 0 1 0
- joint RR_calf_joint: axis 0 -1 0 -> 0 1 0
- joint RR_thigh_joint: axis 0 -1 0 -> 0 1 0
